File: 8x8matrix/8x8matrix_tlc4.brd (EAGLE design)
At the start: 60.4 x 60.5 mm, 6 parts

Commit message: eagle 7
Connections:
- net GND: now also JP2.4; no longer JP2.5
- net N$25: now also JP2.5; no longer JP2.4
Routing:
- net N$25: track 26.2 -> 25.1 mm
Changed lines of the file:
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@@
 <?xml version="1.0" encoding="utf-8"?>
 <!DOCTYPE eagle SYSTEM "eagle.dtd">
-<eagle version="6.5.0">
+<eagle version="7.1.0">
 <drawing>
 <settings>
@@
 <layer number="17" name="Pads" color="2" fill="1" visible="yes" active="yes"/>
 <layer number="18" name="Vias" color="2" fill="1" visible="yes" active="yes"/>
-<layer number="19" name="Unrouted" color="6" fill="1" visible="no" active="yes"/>
+<layer number="19" name="Unrouted" color="6" fill="1" visible="yes" active="yes"/>
 <layer number="20" name="Dimension" color="15" fill="1" visible="yes" active="yes"/>
 <layer number="21" name="tPlace" color="7" fill="1" visible="no" active="yes"/>
-<layer number="22" name="bPlace" color="7" fill="1" visible="no" active="yes"/>
+<layer number="22" name="bPlace" color="7" fill="1" visible="yes" active="yes"/>
 <layer number="23" name="tOrigins" color="15" fill="1" visible="yes" active="yes"/>
 <layer number="24" name="bOrigins" color="15" fill="1" visible="yes" active="yes"/>
@@
 <layer number="35" name="tGlue" color="7" fill="4" visible="no" active="yes"/>
 <layer number="36" name="bGlue" color="7" fill="5" visible="no" active="yes"/>
-<layer number="37" name="tTest" color="7" fill="1" visible="no" active="yes"/>
-<layer number="38" name="bTest" color="7" fill="1" visible="no" active="yes"/>
+<layer number="37" name="tTest" color="7" fill="1" visible="yes" active="yes"/>
+<layer number="38" name="bTest" color="7" fill="1" visible="yes" active="yes"/>
 <layer number="39" name="tKeepout" color="4" fill="11" visible="no" active="yes"/>
 <layer number="40" name="bKeepout" color="1" fill="11" visible="no" active="yes"/>
@@
 <layer number="49" name="Reference" color="7" fill="1" visible="no" active="yes"/>
 <layer number="50" name="dxf" color="7" fill="1" visible="no" active="no"/>
-<layer number="51" name="tDocu" color="7" fill="1" visible="no" active="yes"/>
-<layer number="52" name="bDocu" color="7" fill="1" visible="no" active="yes"/>
+<layer number="51" name="tDocu" color="7" fill="1" visible="yes" active="yes"/>
+<layer number="52" name="bDocu" color="7" fill="1" visible="yes" active="yes"/>
 <layer number="53" name="tGND_GNDA" color="7" fill="9" visible="no" active="no"/>
 <layer number="54" name="bGND_GNDA" color="1" fill="9" visible="no" active="no"/>
@@
 <pass name="Default">
 <param name="RoutingGrid" value="50mil"/>
+<param name="AutoGrid" value="1"/>
+<param name="Efforts" value="0"/>
+<param name="TopRouterVariant" value="1"/>
 <param name="tpViaShape" value="round"/>
 <param name="PrefDir.1" value="|"/>
@@
 <contactref element="U$9" pad="4"/>
 <contactref element="U$9" pad="5"/>
-<contactref element="JP2" pad="5"/>
 <contactref element="R2" pad="2"/>
 <contactref element="R2" pad="1"/>
+<contactref element="JP2" pad="4"/>
 <wire x1="47.368" y1="39.243" x2="50.168" y2="39.243" width="0" layer="19" extent="16-16"/>
-<wire x1="30.226" y1="30.226" x2="36.664" y2="35.941" width="0" layer="19" extent="16-16"/>
 </signal>
 <signal name="5.0V">
@@
 <signal name="N$25">
 <contactref element="U$14" pad="30"/>
-<contactref element="JP2" pad="4"/>
 <wire x1="33.801" y1="34.176" x2="33.801" y2="33.509" width="0.4064" layer="16"/>
 <wire x1="33.801" y1="33.509" x2="34.0741" y2="33.2359" width="0.4064" layer="16"/>
-<wire x1="56.896" y1="27.686" x2="41.656" y2="27.686" width="0.4064" layer="16"/>
-<wire x1="41.656" y1="27.686" x2="36.0807" y2="33.2359" width="0.4064" layer="16"/>
 <wire x1="36.0807" y1="33.2359" x2="34.0741" y2="33.2359" width="0.4064" layer="16"/>
+<contactref element="JP2" pad="5"/>
+<wire x1="36.0807" y1="33.2359" x2="39.0906" y2="30.226" width="0.4064" layer="16"/>
+<wire x1="39.0906" y1="30.226" x2="56.896" y2="30.226" width="0.4064" layer="16"/>
 </signal>
 <signal name="N$1">
