File: 8x8matrix/8x8matrix_tlc4.sch (EAGLE design)
At the start: 6 parts

Commit message: eagle 7
Connections:
- net GND: now also JP2.4; no longer JP2.5
- net N$25: now also JP2.5; no longer JP2.4
Changed lines of the file:
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@@
 <?xml version="1.0" encoding="utf-8"?>
 <!DOCTYPE eagle SYSTEM "eagle.dtd">
-<eagle version="6.5.0">
+<eagle version="7.1.0">
 <drawing>
 <settings>
@@
 <part name="U$6" library="microbuilder" deviceset="5.0V" device=""/>
 <part name="U$8" library="microbuilder" deviceset="GND" device=""/>
-<part name="U$13" library="microbuilder" deviceset="GND" device=""/>
 <part name="U$12" library="microbuilder" deviceset="5.0V" device=""/>
 <part name="U$14" library="TLC5947" deviceset="TLC5947" device="DAP"/>
@@
 <part name="U$11" library="microbuilder" deviceset="GND" device=""/>
 <part name="U$15" library="microbuilder" deviceset="GND" device=""/>
+<part name="U$16" library="microbuilder" deviceset="GND" device=""/>
 </parts>
 <sheets>
@@
 <attribute name="VALUE" x="-9.144" y="135.89" size="1.27" layer="96"/>
 </instance>
-<instance part="U$13" gate="G$1" x="-48.26" y="142.24" rot="R90"/>
 <instance part="U$12" gate="G$1" x="-48.26" y="144.78" rot="R270"/>
 <instance part="U$14" gate="G$1" x="10.16" y="157.48"/>
@@
 <instance part="U$11" gate="G$1" x="0" y="111.76" rot="R90"/>
 <instance part="U$15" gate="G$1" x="-15.24" y="111.76" rot="R270"/>
+<instance part="U$16" gate="G$1" x="-48.26" y="139.7" rot="R90"/>
 </instances>
 <busses>
@@
 </segment>
 <segment>
-<pinref part="U$13" gate="G$1" pin="GND"/>
-<pinref part="JP2" gate="G$1" pin="5"/>
-</segment>
-<segment>
 <pinref part="R2" gate="G$1" pin="2"/>
 <pinref part="U$11" gate="G$1" pin="GND"/>
@@
 <pinref part="R2" gate="G$1" pin="1"/>
 <pinref part="U$15" gate="G$1" pin="GND"/>
+</segment>
+<segment>
+<pinref part="JP2" gate="G$1" pin="4"/>
+<pinref part="U$16" gate="G$1" pin="GND"/>
 </segment>
 </net>
@@
 <net name="N$25" class="0">
 <segment>
-<wire x1="-50.8" y1="139.7" x2="-25.4" y2="139.7" width="0.1524" layer="91"/>
 <pinref part="U$14" gate="G$1" pin="XLAT"/>
-<wire x1="-25.4" y1="139.7" x2="-25.4" y2="144.78" width="0.1524" layer="91"/>
+<wire x1="-25.4" y1="142.24" x2="-25.4" y2="144.78" width="0.1524" layer="91"/>
 <wire x1="-25.4" y1="144.78" x2="-7.62" y2="144.78" width="0.1524" layer="91"/>
-<pinref part="JP2" gate="G$1" pin="4"/>
-</segment>
-</net>
+<pinref part="JP2" gate="G$1" pin="5"/>
+<wire x1="-50.8" y1="142.24" x2="-25.4" y2="142.24" width="0.1524" layer="91"/>
+</segment>
+</net>
