File: 8x8matrix/8x8matrix.sch (EAGLE design)
At the start: 18 parts

Commit message: changed 238 to 138
Parts:
- U$9: value CD74HC238M -> 74HC138D; device mylib:CD74HC238M -> mylib:74HC138D
Changed lines of the file:
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@@
 <part name="U$2" library="microbuilder" deviceset="GND" device=""/>
 <part name="U$3" library="microbuilder" deviceset="GND" device=""/>
-<part name="U$9" library="mylib" deviceset="CD74HC238" device="M"/>
+<part name="U$9" library="mylib" deviceset="74HC138" device="D"/>
 <part name="U$7" library="microbuilder" deviceset="5.0V" device=""/>
 <part name="U$10" library="microbuilder" deviceset="GND" device=""/>
