File: 8x8matrix/8x8matrix.sch (EAGLE design)
At the start: 18 parts

Commit message: added prints
Connections:
- net N$36 renamed A0
- net N$37 renamed A1
- net N$38 renamed A2
Changed lines of the file:
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@@
 </segment>
 </net>
-<net name="N$36" class="0">
+<net name="A0" class="0">
 <segment>
 <pinref part="U$9" gate="G$1" pin="A0"/>
@@
 </segment>
 </net>
-<net name="N$37" class="0">
+<net name="A1" class="0">
 <segment>
 <pinref part="U$9" gate="G$1" pin="A1"/>
@@
 </segment>
 </net>
-<net name="N$38" class="0">
+<net name="A2" class="0">
 <segment>
 <pinref part="U$9" gate="G$1" pin="A2"/>
